File: Hardware/Source/Primer_esquematico.kicad_pcb (KiCad board)
At the start: 2 copper layers, 108 x 25 mm, 6 parts, among them J2 Screw_Terminal_01x06, SW1 SW_Push, U1 XIAO-ESP32-C3-DIP, U3 2472, U4 MICRO SD

Commit message: Actualización de pcb
Se adjunta el diseño final del PCB, el cual ha sido enviado a producción conforme a las especificaciones técnicas requeridas.
Parts:
- removed U4: MICRO SD, Mis_creaciones:Targeta USB mini
- added ?: , , F.Cu at (246.0, 89.0)
- added ?: , , F.Cu at (246.0, 72.0)
- added J1: Screw_Terminal_01x06, Mis_creaciones:Conector_flex, F.Cu at (221.5, 67.8)
- added R1: R_Small_US, Resistor_THT:R_Axial_DIN0204_L3.6mm_D1.6mm_P1.90mm_Vertical, F.Cu at (218.9, 108.8)
- added R2: R_Small_US, Resistor_THT:R_Axial_DIN0204_L3.6mm_D1.6mm_P1.90mm_Vertical, F.Cu at (216.0, 108.7)
- added REF**: MountingHole_2.2mm_M2_DIN965_Pad, MountingHole:MountingHole_2.2mm_M2_DIN965_Pad, F.Cu at (246.0, 97.0)
- added REF**: MountingHole_2.2mm_M2_DIN965_Pad, MountingHole:MountingHole_2.2mm_M2_DIN965_Pad, F.Cu at (173.0, 115.0)
- added REF**: MountingHole_2.2mm_M2_DIN965_Pad, MountingHole:MountingHole_2.2mm_M2_DIN965_Pad, F.Cu at (246.0, 115.0)
- added REF**: MountingHole_2.2mm_M2_DIN965_Pad, MountingHole:MountingHole_2.2mm_M2_DIN965_Pad, F.Cu at (173.0, 97.0)
- added U2: GY-521, GY-521:MODULE_GY-521, F.Cu at (240.0, 80.5)
- added U5: ~, Mis_creaciones:Conector_bateria_xiao, F.Cu at (208.4, 113.0)
- moved U3 43.0 mm to (199.9, 105.7)
- moved J2 41.5 mm to (189.6, 116.6)
Connections:
- U1 pad 1: unconnected-(U1-GPIO2_A0_D0-Pad1) -> Net-(U1-GPIO2_A0_D0)
- U1 pad 10: Net-(U1-GPIO9_D9_MISO) -> unconnected-(U1-GPIO9_D9_MISO-Pad10)
- U1 pad 11: Net-(U1-GPIO10_D10_MOSI) -> unconnected-(U1-GPIO10_D10_MOSI-Pad11)
- U1 pad 3: Net-(U1-GPIO4_A2_D2) -> unconnected-(U1-GPIO4_A2_D2-Pad3)
- U1 pad 9: Net-(U1-GPIO8_D8_SCK) -> unconnected-(U1-GPIO8_D8_SCK-Pad9)
Routing:
- net GND: track 169.0 -> 89.3 mm
- net Net-(U1-GPIO4_A2_D2): track 78.0 -> 0.00 mm
- net Net-(J2-Pin_5): track 132.9 -> 68.4 mm
- net Net-(J2-Pin_1): track 107.6 -> 59.9 mm
- net Net-(J2-Pin_4): track 112.9 -> 73.5 mm
- net Net-(U1-GPIO8_D8_SCK): track 34.6 -> 0.00 mm
- net Net-(U1-GPIO2_A0_D0): track 0.00 -> 29.3 mm
- net Net-(U1-GPIO10_D10_MOSI): track 26.6 -> 0.00 mm
- net Net-(U1-GPIO9_D9_MISO): track 24.3 -> 0.00 mm
- net Net-(J1-Pin_3): track 0.00 -> 13.6 mm
- net Net-(J1-Pin_5): track 0.00 -> 5.65 mm
- net Net-(J1-Pin_4): track 0.00 -> 5.65 mm
- net Net-(J1-Pin_1): track 0.00 -> 4.59 mm
- net Net-(J1-Pin_2): track 0.00 -> 4.59 mm
- net Net-(U5--2): track 0.00 -> 4.53 mm
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- added copper zone on F.Cu, net (none)
Other:
- board size 108 x 25 mm -> 80 x 50 mm
- board text added: "CDIO 3"
- board text added: "Emerson, Joseph, Rodrigo"
- board text added: "LANCEA"
